Commit message: feat: harden protocol-v3 grasp execution

File: src/real-arm/alicia_d_descriptions/urdf/alicia_duo_with_gripper.urdf (robot description, URDF)
Before this commit: robot alicia_D_v5_5, 11 links, 10 joints
Joints:
- joint left_finger: axis 0 0 1 -> 0 0 -1; origin xyz=-0.0002 0.050502 0.13118 rpy=-1.5708 0 0 -> xyz=-0.0002 0.000502 0.131180183660255 rpy=-1.5708 0 0
- joint right_finger: axis 0 0 -1 -> 0 0 1; origin xyz=-0.0002 -0.050498 0.13118 rpy=1.5708 0 0 -> xyz=-0.0002 -0.000498 0.131180183660255 rpy=1.5708 0 0
